File: EuroClockMD/EuroClockMD-Panel.kicad_pcb (KiCad board)
At the start: 2 copper layers, 30 x 128.5 mm, 12 parts

Commit message: retraced EuroClockMD-Pin and moved holes in EuroClockMD-panel
Parts:
- moved REF** 1.34 mm to (227.2, 153.4)
- moved REF** 1.30 mm to (211.9, 30.9)
