File: EuroClockMD/EuroClockMD.kicad_pcb (KiCad board)
At the start: 2 copper layers, 33 parts, among them J1 AudioJack2_SwitchT (Gate Out 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, J2 AudioJack2_SwitchT (Gate Out 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, J3 AudioJack2_SwitchT (Master Cl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, J4 AudioJack2_SwitchT (External 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, J5 EURO_PWR_2x5, SW1 SW_SPDT (Internal Pullup)

Commit message: update
Parts:
- added J6: Conn_01x15_Pin_Left, Connector_PinHeader_2.54mm:PinHeader_1x15_P2.54mm_Vertical, F.Cu at (168.9, 45.7)
- added J7: Conn_01x15_Socket_Left, Connector_PinSocket_2.54mm:PinSocket_1x15_P2.54mm_Vertical, B.Cu at (130.5, 45.7)
- added J8: Conn_01x15_Socket_Right, Connector_PinSocket_2.54mm:PinSocket_1x15_P2.54mm_Vertical, B.Cu at (153.4, 45.7)
- added J9: Conn_01x15_Pin_Right, Connector_PinHeader_2.54mm:PinHeader_1x15_P2.54mm_Vertical, F.Cu at (191.8, 45.7)
- A1, D1, D10, D11, D12, D3, D4, D5, D7, D8, J5: moved to B.Cu
- C1, C2: footprint Capacitor_THT:CP_Axial_L10.0mm_D6.0mm_P15.00mm_Horizontal -> Capacitor_THT:C_Disc_D3.0mm_W1.6mm_P2.50mm; moved to B.Cu
- D2: value LED -> GATE OUT 1 LED; footprint LED_THT:LED_D3.0mm -> LED_THT:LED_D5.0mm
- D6: value LED -> GATE OUT 2 LED; footprint LED_THT:LED_D3.0mm -> LED_THT:LED_D5.0mm
- D9: value LED -> CLOCK OUT LED; footprint LED_THT:LED_D3.0mm -> LED_THT:LED_D5.0mm
- J1: value AudioJack2_SwitchT (Gate Out 1) -> GATE OUT 1
- J2: value AudioJack2_SwitchT (Gate Out 2) -> GATE OUT 2
- J3: value AudioJack2_SwitchT (Master Clock Out) -> CLOCK OUT
- J4: value AudioJack2_SwitchT (External Clock In) -> EXT CLK IN
- R1, R10, R2, R3, R4, R5, R6, R7, R8, R9: footprint Resistor_THT:R_Axial_DIN0207_L6.3mm_D2.5mm_P10.16mm_Horizontal -> Resistor_THT:R_Axial_DIN0207_L6.3mm_D2.5mm_P7.62mm_Horizontal; moved to B.Cu
- RV1: value 100K (Multi/Div) -> 100K MULTI/DIV
- RV2: value 100K (Rate) -> 100K RATE
- SW1: footprint TerminalBlock:TerminalBlock_bornier-3_P5.08mm -> Button_Switch_THT:SW_Slide-03_Wuerth-WS-SLTV_10x2.5x6.4_P2.54mm
- moved A1 112.8 mm to (172.7, 81.3)
- moved J2 101.1 mm to (148.3, 135.8)
- moved R10 96.8 mm to (176.5, 124.5)
- moved J1 94.4 mm to (148.3, 120.6)
- moved D4 93.3 mm to (184.2, 114.3), turned to 180 degrees
- moved D10 90.2 mm to (184.2, 119.4), turned to 180 degrees
- moved D1 88.0 mm to (184.2, 88.9), turned to 180 degrees
- moved J5 87.7 mm to (175.3, 137.2), turned to -90 degrees
- moved R5 87.5 mm to (139.4, 142.2), turned to 180 degrees
- moved D3 85.7 mm to (176.5, 109.2)
- moved D11 85.3 mm to (176.5, 129.5)
- moved C1 84.7 mm to (142.0, 55.9), turned to -90 degrees
- moved C2 82.2 mm to (145.8, 82.6), turned to -90 degrees
- moved D8 80.0 mm to (176.5, 104.1)
- moved D7 79.8 mm to (176.5, 99.1)
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Connections:
- A1 pad 10: Net-(A1-D7) -> P5
- A1 pad 11: Net-(A1-D8) -> P6
- A1 pad 14: Net-(A1-D11) -> P4
- A1 pad 22: Net-(A1-A3) -> P1
- A1 pad 23: Net-(A1-A4) -> P2
- A1 pad 27: 5V -> P5V
- A1 pad 6: Net-(A1-D3) -> P3
- C1 pad 1: Net-(A1-A3) -> (no net)
- C1 pad 2: GND -> (no net)
- C2 pad 1: Net-(A1-A4) -> (no net)
- C2 pad 2: GND -> (no net)
- D1 pad 1: 5V -> P5V
- D1 pad 2: Net-(A1-D8) -> P6
- D10 pad 1: 5V -> P5V
- D10 pad 2: Net-(A1-D3) -> P3
- D11 pad 1: Net-(A1-D3) -> P3
- D12 pad 1: GND -> (no net)
- D12 pad 2: Net-(A1-D3) -> (no net)
- D2 pad 1: GND -> (no net)
- D2 pad 2: Net-(D2-A) -> (no net)
- D3 pad 1: Net-(A1-D7) -> P5
- D4 pad 1: 5V -> P5V
- D4 pad 2: Net-(A1-D7) -> P5
- D5 pad 1: Net-(A1-D8) -> P6
- D6 pad 1: GND -> (no net)
- D6 pad 2: Net-(D6-A) -> (no net)
- D7 pad 1: Net-(D7-K) -> P7
- D8 pad 1: Net-(D7-K) -> P7
- D9 pad 1: GND -> (no net)
- D9 pad 2: unconnected-(D9-A-Pad2) -> (no net)
- J1 pad S: GND -> (no net)
- J1 pad T: Net-(J1-PadT) -> (no net)
- J1 pad TN: unconnected-(J1-PadTN) -> (no net)
- J2 pad S: GND -> (no net)
- J2 pad T: Net-(J2-PadT) -> (no net)
- J2 pad TN: unconnected-(J2-PadTN) -> (no net)
- J3 pad S: unconnected-(J3-PadS) -> (no net)
- J3 pad T: GND -> (no net)
- J3 pad TN: unconnected-(J3-PadTN) -> (no net)
- J4 pad S: GND -> (no net)
- J4 pad T: Net-(J4-PadT) -> (no net)
- J4 pad TN: unconnected-(J4-PadTN) -> (no net)
- J5 pad 10: unconnected-(J5--12V-Pad10) -> Net-(A1-VIN)
- J5 pad 2: Net-(A1-VIN) -> unconnected-(J5--12V-Pad2)
- J5 pad 9: unconnected-(J5--12V-Pad9) -> Net-(A1-VIN)
- R1 pad 1: Net-(R1-Pad1) -> (no net)
- R1 pad 2: Net-(A1-A3) -> (no net)
- R10 pad 1: Net-(A1-D3) -> P3
- R2 pad 1: Net-(D2-A) -> (no net)
- R2 pad 2: Net-(A1-D7) -> (no net)
- R3 pad 1: Net-(A1-D7) -> (no net)
- R3 pad 2: Net-(J1-PadT) -> (no net)
- R4 pad 1: Net-(D7-K) -> (no net)
- R4 pad 2: GND -> (no net)
- R5 pad 1: Net-(D6-A) -> (no net)
- R5 pad 2: Net-(A1-D8) -> (no net)
- R6 pad 1: Net-(R6-Pad1) -> (no net)
- R6 pad 2: Net-(A1-A4) -> (no net)
- R7 pad 1: Net-(A1-D8) -> (no net)
- R7 pad 2: Net-(J2-PadT) -> (no net)
- R8 pad 1: unconnected-(R8-Pad1) -> (no net)
- R8 pad 2: GND -> (no net)
- R9 pad 1: Net-(J4-PadT) -> (no net)
- R9 pad 2: Net-(A1-D3) -> (no net)
- RV1 pad 1: 5V -> (no net)
- RV1 pad 2: Net-(R1-Pad1) -> (no net)
- RV1 pad 3: GND -> (no net)
- RV2 pad 1: 5V -> (no net)
- RV2 pad 2: Net-(R6-Pad1) -> (no net)
- RV2 pad 3: GND -> (no net)
- SW1 pad 1: Net-(A1-D11) -> (no net)
- SW1 pad 2: GND -> (no net)
- SW1 pad 3: unconnected-(SW1-C-Pad3) -> (no net)
Routing:
- net (no net): track 0.00 -> 748.7 mm
- net GND: track 0.00 -> 87.1 mm
- net P3: track 0.00 -> 86.0 mm
- net Net-(A1-VIN): track 0.00 -> 63.7 mm
- net P5: track 0.00 -> 62.7 mm
- net Net-(A1-D13): track 0.00 -> 57.6 mm
- net P5V: track 0.00 -> 52.0 mm
- net P7: track 0.00 -> 46.3 mm
- net P6: track 0.00 -> 43.5 mm
- net P4: track 0.00 -> 3.81 mm
- net P2: track 0.00 -> 3.81 mm
- net P1: track 0.00 -> 3.81 mm
Other:
- board outline added: 110.7 x 128.5 mm
- board text added: "CLK IN"
- board text added: "CLK OUT"
- board text added: "GATE OUT 2"
- board text added: "JLCJLCJLCJLC"
- board text added: "MULTI/DIV"
- board text added: "ORIGINAL DESIGN BY HAGIWO"
- board text added: "RATE"
- board text added: "SynthLab"
- board text added: "TIME MANAGEMENT"
- board text added: "V1.0 PCBs + PANEL BY 42 BERLIN SYNTHLAB https://github.com/fablabnk/SynthLabProjects"

Commit message: retraced EuroClockMD-Pin and moved holes in EuroClockMD-panel
Parts:
- added REF**: MountingHole_4.5mm, MountingHole:MountingHole_4.5mm, F.Cu at (160.5, 143.3)
- added REF**: MountingHole_6mm, Library:MountingHole_6mm, F.Cu at (173.2, 128.1)
- added REF**: MountingHole_6mm, Library:MountingHole_6mm, F.Cu at (166.9, 77.3)
- added REF**: MountingHole_4.5mm, MountingHole:MountingHole_4.5mm, F.Cu at (173.2, 97.6)
- added REF**: MountingHole_6mm, Library:MountingHole_6mm, F.Cu at (173.2, 112.8)
- added REF**: MountingHole_6mm, Library:MountingHole_6mm, F.Cu at (160.5, 97.6)
- added REF**: Eurorack_Panel_ScrewHole_Oval, Library:Eurorack_Panel_ScrewHole_Oval, F.Cu at (159.1, 35.8)
- added REF**: MountingHole_6mm, Library:MountingHole_6mm, F.Cu at (173.2, 143.3)
- added REF**: MountingHole_4.5mm, MountingHole:MountingHole_4.5mm, F.Cu at (160.5, 128.1)
- added REF**: Eurorack_Panel_ScrewHole_Oval, Library:Eurorack_Panel_ScrewHole_Oval, F.Cu at (174.4, 158.4)
- added REF**: MountingHole_6mm, Library:MountingHole_6mm, F.Cu at (166.9, 51.9)
- added REF**: MountingHole_6mm, Library:MountingHole_6mm, F.Cu at (160.5, 112.8)
- J5: footprint Connector_IDC:IDC-Header_2x05_P2.54mm_Vertical -> 4ms_Connector:Pins_2x05_2.54mm_TH_EurorackPower_Shrouded
- moved J1 121.2 mm to (269.3, 127.8)
- moved J2 121.2 mm to (269.3, 143.0)
- moved J3 121.2 mm to (269.3, 112.5)
- moved RV1 121.2 mm to (263.0, 51.7)
- moved RV2 121.2 mm to (263.0, 77.1)
- moved C1 121.2 mm to (262.9, 63.1)
- moved C2 121.2 mm to (266.7, 89.8)
- moved D12 121.2 mm to (262.9, 145.6)
- moved D2 121.2 mm to (255.3, 127.8)
- moved D6 121.2 mm to (255.3, 143.0)
- moved J7 121.2 mm to (251.5, 52.9)
- moved J8 121.2 mm to (274.4, 52.9)
- moved R1 121.2 mm to (270.5, 60.5)
- moved R2 121.2 mm to (262.9, 117.6)
- moved R3 121.2 mm to (262.9, 127.8)
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Routing:
- net GND: track 87.1 -> 0.00 mm
- net Net-(A1-VIN): track 63.7 -> 0.00 mm
- net P3: track 86.0 -> 67.9 mm
- net P7: track 46.3 -> 48.2 mm
- net Net-(A1-D13): track 57.6 -> 56.1 mm
- added copper zone on B.Cu, net GND
- added copper zone on F.Cu, net Net-(A1-VIN)
Other:
- board size 110.7 x 128.5 mm -> 202.3 x 128.5 mm
